Commit message: Add chin-mounted 3D lidar sensor (gpu_lidar with vertical scan)
Adds a new fixed link/joint (chin_lidar_frame) off base_link plus a
gpu_lidar sensor with a vertical scan block, mirroring the existing
laser/imu/camera sensor pattern, and bridges the point cloud topic
via ros_gz_bridge (PointCloud2 <-> gz.msgs.PointCloudPacked).

Mount offset/pitch and vertical FOV are placeholder estimates (based
on the unused go2_description.urdf's Head_lower reference and a
generic 16-channel 3D lidar), not verified real hardware dimensions.

File: go2_description/xacro/gazebo.xacro (robot description, xacro)
@@ -125,4 +125,36 @@
             </sensor>
         </gazebo>
+        <!--
+            顎搭載3D LiDAR。channels/FOVはこのリポジトリ内に実機スペックの根拠がないため、
+            一般的な小型3D LiDAR相当(16ch、垂直±15°)を仮値として置いている。
+            実機LiDARの型番が決まり次第、samples/min_angle/max_angleを実スペックに合わせて更新すること。
+        -->
+        <gazebo reference="chin_lidar_frame">
+            <sensor name="chin_lidar" type="gpu_lidar">
+                <pose> 0 0 0 0 0 0 </pose>
+                <visualize>false</visualize>
+                <update_rate>10</update_rate>
+                <lidar>
+                    <scan>
+                        <horizontal>
+                            <samples>360</samples>
+                            <min_angle>-3.14</min_angle>
+                            <max_angle>3.14</max_angle>
+                        </horizontal>
+                        <vertical>
+                            <samples>16</samples>
+                            <min_angle>-0.2618</min_angle>
+                            <max_angle>0.2618</max_angle>
+                        </vertical>
+                    </scan>
+                    <range>
+                        <min>0.05</min>
+                        <max>12</max>
+                    </range>
+                </lidar>
+                <topic>/${robot_name}/chin_lidar/scan</topic>
+                <gz_frame_id>chin_lidar_frame</gz_frame_id>
+            </sensor>
+        </gazebo>
         <gazebo reference="camera_face">
             <!-- <material>Gazebo/Black</material> -->

File: go2_description/xacro/robot.xacro (robot description, xacro)
@@ -82,4 +82,35 @@
         </collision>
     </link>
+    <!--
+        顎(chin)搭載3D LiDAR用フレーム。船内部材ナビゲーション計画(docs/計画_経路生成.md)の
+        「顎LiDARは前下方のみ視野」に対応するダミーリンク。
+        搭載位置(xyz)はこのリポジトリに実機の顎LiDAR寸法が無いため、未使用の
+        go2_description.urdf内のHead_lower(頭部下側)リンクのオフセットを流用した仮値であり、
+        実機の正確な搭載位置を計測でき次第、更新すること。ピッチ角(前下方視野)も仮値。
+    -->
+    <joint name="chin_lidar_joint" type="fixed">
+        <parent link="base_link"/>
+        <child link="chin_lidar_frame"/>
+        <origin xyz="0.29 0.0 -0.06" rpy="0 0.35 0"/>
+    </joint>
+    <link name="chin_lidar_frame">
+        <inertial>
+            <mass value="0.001"/>
+            <origin rpy="0 0 0" xyz="0 0 0"/>
+            <inertia ixx="0.0001" ixy="0" ixz="0" iyy="0.0001" iyz="0" izz="0.0001"/>
+        </inertial>
+        <visual>
+            <origin rpy="0 0 0" xyz="0 0 0"/>
+            <geometry>
+                <cylinder length="0.02" radius="0.02" />
+            </geometry>
+        </visual>
+        <collision>
+            <origin rpy="0 0 0" xyz="0 0 0"/>
+            <geometry>
+                <cylinder length="0.02" radius="0.02" />
+            </geometry>
+        </collision>
+    </link>
     <joint name="imu_joint" type="fixed">
         <parent link="base_link"/>

Commit message: Mount D1-T arm on Go2's rear (placeholder static TF) via ros2_control
- robot.xacro: include d1_arm.xacro and instantiate it as a fixed joint
  off the trunk link. The mount xyz/rpy is an unmeasured placeholder
  (top-rear of trunk) pending the real static TF once hardware arrives.
- gazebo.xacro: add a separate ros2_control <system> block for the 8
  D1 joints, using the same gz_ros2_control/GazeboSimSystem plugin as
  the legs but kept independent so it can't affect leg joint commands.
- ros_control.yaml / gazebo_multi_nav2_world.launch.py: add a
  d1_arm_controller (position_controllers/JointGroupPositionController)
  and its spawner, separate from the legs' joint_group_controller.

Verified: colcon build clean, xacro renders the combined URDF with all
9 d1_ joints/links correctly parented under trunk (check_urdf), gz sdf
conversion has no d1-related warnings, and the model spawns in a
headless gz sim with all d1_link* entities present.

Go2_deploy Issue #65.

File: go2_description/xacro/gazebo.xacro (robot description, xacro)
@@ -82,4 +82,61 @@
             </joint>
             <joint name="rh_lower_leg_joint">
+                <command_interface name="position"/>
+                <state_interface name="position"/>
+                <state_interface name="velocity"/>
+                <state_interface name="effort"/>
+            </joint>
+        </ros2_control>
+        <!--
+            D1-Tアーム用のros2_control(脚用GazeboSystemとは別系統。歩行制御の
+            joint_group_controllerを巻き込まないよう、コントローラを分離している)。
+        -->
+        <ros2_control name="${robot_name}_D1ArmGazeboSystem" type="system">
+            <hardware>
+                <plugin>gz_ros2_control/GazeboSimSystem</plugin>
+            </hardware>
+            <joint name="d1_joint1">
+                <command_interface name="position"/>
+                <state_interface name="position"/>
+                <state_interface name="velocity"/>
+                <state_interface name="effort"/>
+            </joint>
+            <joint name="d1_joint2">
+                <command_interface name="position"/>
+                <state_interface name="position"/>
+                <state_interface name="velocity"/>
+                <state_interface name="effort"/>
+            </joint>
+            <joint name="d1_joint3">
+                <command_interface name="position"/>
+                <state_interface name="position"/>
+                <state_interface name="velocity"/>
+                <state_interface name="effort"/>
+            </joint>
+            <joint name="d1_joint4">
+                <command_interface name="position"/>
+                <state_interface name="position"/>
+                <state_interface name="velocity"/>
+                <state_interface name="effort"/>
+            </joint>
+            <joint name="d1_joint5">
+                <command_interface name="position"/>
+                <state_interface name="position"/>
+                <state_interface name="velocity"/>
+                <state_interface name="effort"/>
+            </joint>
+            <joint name="d1_joint6">
+                <command_interface name="position"/>
+                <state_interface name="position"/>
+                <state_interface name="velocity"/>
+                <state_interface name="effort"/>
+            </joint>
+            <joint name="d1_joint_l">
+                <command_interface name="position"/>
+                <state_interface name="position"/>
+                <state_interface name="velocity"/>
+                <state_interface name="effort"/>
+            </joint>
+            <joint name="d1_joint_r">
                 <command_interface name="position"/>
                 <state_interface name="position"/>

File: go2_description/xacro/robot.xacro (robot description, xacro)
@@ -7,4 +7,5 @@
     <!-- <xacro:include filename="$(find go2_description)/xacro/stairs.xacro"/> -->
     <xacro:include filename="$(find go2_description)/xacro/gazebo.xacro"/>
+    <xacro:include filename="$(find d1_550_description)/urdf/d1_arm.xacro"/>
     <!-- <xacro:include filename="$(find go2_description)/launch/stairs.urdf.xacro"/> -->
     <xacro:robot_gazebo_sensors robot_name="$(arg robot_name)"/>
@@ -57,4 +58,10 @@
         </inertial>
     </link>
+    <!--
+        D1-Tアーム(背面搭載)。mount原点(xyz/rpy)は実機未計測の仮値(trunk上面・後方寄り)。
+        実機到着後にGo2背面への実際の搭載位置を計測し、更新すること
+        (Go2_deploy Issue #65、docs/計画/アーム動作.md §5)。
+    -->
+    <xacro:d1_arm parent="trunk" prefix="d1_" xyz="-0.15 0 0.10" rpy="0 0 0"/>
     <joint name='laser_scan' type='fixed'>
         <parent link="base_link"/>,

Commit message: feat: 🎥 Go2_deploy#85 D1先端にカメラ(RGB・仮の位置)を追加し、/robot1/arm_cam/{image,camera_info}をROSへ橋渡しする

File: go2_description/xacro/gazebo.xacro (robot description, xacro)
@@ -255,4 +255,27 @@
             </sensor>
         </gazebo>
+        <!-- D1 先端のカメラ(実機は RealSense D405、水平視野 約87度)。RGB のみ。深度は未対応(Go2_deploy #85) -->
+        <gazebo reference="d1_arm_cam">
+            <sensor name="arm_camera" type="camera">
+                <pose> 0 0 0 0 0 0 </pose>
+                <visualize>false</visualize>
+                <update_rate>10</update_rate>
+                <camera>
+                    <camera_info_topic>/${robot_name}/arm_cam/camera_info</camera_info_topic>
+                    <horizontal_fov>1.518</horizontal_fov>
+                    <image>
+                        <format>R8G8B8</format>
+                        <width>640</width>
+                        <height>360</height>
+                    </image>
+                    <clip>
+                        <near>0.05</near>
+                        <far>4.0</far>
+                    </clip>
+                </camera>
+                <topic>/${robot_name}/arm_cam/image</topic>
+                <gz_frame_id>d1_arm_cam</gz_frame_id>
+            </sensor>
+        </gazebo>
         <gazebo reference="trunk">
             <mu1>0.2</mu1>

File: go2_description/xacro/robot.xacro (robot description, xacro)
@@ -197,4 +197,19 @@
     </link>
   -->
+    <!-- D1 先端のカメラ(実機は RealSense D405)。見た目(取付金具)は無く、センサの位置だけを置く。
+         **位置・向きは仮の値**(Inventor の設計値が来たら差し替える。Go2_deploy #85)。
+         link6 の +x がグリッパの突き出す向き。そこから少し上・前に置き、+x(グリッパの先)を向ける -->
+    <joint name="d1_arm_cam_joint" type="fixed">
+        <parent link="d1_link6"/>
+        <child link="d1_arm_cam"/>
+        <origin xyz="0.03 0 0.045" rpy="0 0 0"/>
+    </joint>
+    <link name="d1_arm_cam">
+        <inertial>
+            <mass value="0.001"/>
+            <origin rpy="0 0 0" xyz="0 0 0"/>
+            <inertia ixx="0.0001" ixy="0" ixz="0" iyy="0.0001" iyz="0" izz="0.0001"/>
+        </inertial>
+    </link>
     <joint name="camera_face_joint" type="fixed">
         <parent link="base_link"/>

Commit message: fix: 🐛 Go2_deploy#85 レビュー対応(光学フレーム追加・preserveFixedJoint・enable_arm_cam引数・nearをD405最短に・画像はimage_bridge経由に)

File: go2_description/xacro/gazebo.xacro (robot description, xacro)
@@ -255,5 +255,14 @@
             </sensor>
         </gazebo>
-        <!-- D1 先端のカメラ(実機は RealSense D405、水平視野 約87度)。RGB のみ。深度は未対応(Go2_deploy #85) -->
+        <!-- D1 先端のカメラ(実機は RealSense D405、水平視野 約87度)。RGB のみ。深度は未対応(Go2_deploy #85)。
+             near は D405 の最短測距(約7cm)に合わせた。fixed joint はURDF→SDF変換で統合されると
+             フレームが TF から消えるので、preserveFixedJoint で残す -->
+        <xacro:if value="$(arg enable_arm_cam)">
+        <gazebo reference="d1_arm_cam_joint">
+            <preserveFixedJoint>true</preserveFixedJoint>
+        </gazebo>
+        <gazebo reference="d1_arm_cam_optical_joint">
+            <preserveFixedJoint>true</preserveFixedJoint>
+        </gazebo>
         <gazebo reference="d1_arm_cam">
             <sensor name="arm_camera" type="camera">
@@ -270,12 +279,13 @@
                     </image>
                     <clip>
-                        <near>0.05</near>
+                        <near>0.07</near>
                         <far>4.0</far>
                     </clip>
                 </camera>
                 <topic>/${robot_name}/arm_cam/image</topic>
-                <gz_frame_id>d1_arm_cam</gz_frame_id>
+                <gz_frame_id>d1_arm_cam_optical_frame</gz_frame_id>
             </sensor>
         </gazebo>
+        </xacro:if>
         <gazebo reference="trunk">
             <mu1>0.2</mu1>

File: go2_description/xacro/robot.xacro (robot description, xacro)
@@ -212,4 +212,18 @@
         </inertial>
     </link>
+    <!-- 光学フレーム(ROS の画像系: z 前方・x 右・y 下)。画像の frame_id はこちらにする。
+         AprilTag・image_geometry・rviz の Camera 表示は、この向きを前提にしている -->
+    <joint name="d1_arm_cam_optical_joint" type="fixed">
+        <parent link="d1_arm_cam"/>
+        <child link="d1_arm_cam_optical_frame"/>
+        <origin xyz="0 0 0" rpy="${-pi/2} 0 ${-pi/2}"/>
+    </joint>
+    <link name="d1_arm_cam_optical_frame">
+        <inertial>
+            <mass value="0.001"/>
+            <origin rpy="0 0 0" xyz="0 0 0"/>
+            <inertia ixx="0.0001" ixy="0" ixz="0" iyy="0.0001" iyz="0" izz="0.0001"/>
+        </inertial>
+    </link>
     <joint name="camera_face_joint" type="fixed">
         <parent link="base_link"/>
